File: UsbHost_hw/UsbHostLora.kicad_pcb (KiCad board)
At the start: 0 parts

Commit message: Routing done
Parts:
- added ANT1: ANT_PCB_MONO_2PIN, Antennas:Firefly_868, F.Cu at (155.6, 111.6)
- added C1: 2u2, Capacitors:CAP_0603, F.Cu at (148.6, 136.1)
- added C10: 0.1u, Capacitors:CAP_0402, F.Cu at (150.9, 118.9)
- added C11: 1u, Capacitors:CAP_0603, F.Cu at (148.9, 117.9)
- added C12: 0.1u, Capacitors:CAP_0402, F.Cu at (147.7, 139.0)
- added C13: 0.1u, Capacitors:CAP_0402, F.Cu at (145.9, 135.7)
- added C14: 10n, Capacitors:CAP_0402, F.Cu at (150.4, 96.6)
- added C15: 47pF, Capacitors:CAP_0402, F.Cu at (150.4, 95.5)
- added C16: 1.5pF, Capacitors:CAP_0402, F.Cu at (149.9, 89.4)
- added C17: 22pF, Capacitors:CAP_0402, F.Cu at (148.6, 93.8)
- added C18: 8.2pF, Capacitors:CAP_0402, F.Cu at (146.8, 94.3)
- added C19: 8.2pF, Capacitors:CAP_0402, F.Cu at (146.8, 90.0)
- added C2: 18pF, Capacitors:CAP_0603, F.Cu at (153.8, 113.8)
- added C20: 3.3pF, Capacitors:CAP_0402, F.Cu at (146.8, 88.8)
- added C21: 47pF, Capacitors:CAP_0402, F.Cu at (149.3, 84.0)
- added C22: 47pF, Capacitors:CAP_0402, F.Cu at (154.5, 94.5)
- added C23: C, Capacitors:CAP_0402, F.Cu at (151.1, 82.3)
- added C24: C, Capacitors:CAP_0402, F.Cu at (147.5, 81.3)
- added C25: 3.3pF, Capacitors:CAP_0402, F.Cu at (154.6, 96.2)
- added C26: 1000pF, Capacitors:CAP_0402, F.Cu at (151.1, 85.9)
- added C27: 1000pF, Capacitors:CAP_0402, F.Cu at (147.5, 85.9)
- added C28: 0.1u, Capacitors:CAP_0402, F.Cu at (145.2, 100.8)
- added C29: 0.1u, Capacitors:CAP_0402, F.Cu at (153.2, 105.8)
- added C3: 18pF, Capacitors:CAP_0603, F.Cu at (150.7, 116.2)
- added C30: 0.1u, Capacitors:CAP_0402, F.Cu at (152.5, 95.5)
- added C31: 47pF, Capacitors:CAP_0402, F.Cu at (152.5, 96.6)
- added C32: 0.1u, Capacitors:CAP_0402, F.Cu at (145.2, 99.1)
- added C33: 0.1u, Capacitors:CAP_0402, F.Cu at (145.2, 101.9)
- added C34: 18pF, Capacitors:CAP_0603, F.Cu at (144.2, 108.6)
- added C35: 18pF, Capacitors:CAP_0603, F.Cu at (143.2, 101.0)
- added C4: 10u, Capacitors:CAP_0603, F.Cu at (158.4, 118.0)
- added C5: 0.1u, Capacitors:CAP_0402, F.Cu at (145.4, 123.8)
- added C6: 0.1u, Capacitors:CAP_0402, F.Cu at (145.4, 130.3)
- added C7: 0.1u, Capacitors:CAP_0402, F.Cu at (156.6, 134.5)
- added C8: 0.1u, Capacitors:CAP_0402, F.Cu at (160.9, 123.3)
- added C9: 0.1u, Capacitors:CAP_0402, F.Cu at (156.9, 118.5)
- added DA1: MCP1700, SOT:SOT23-3A, F.Cu at (145.3, 138.5)
- added DA2: PE4259, SOT:SC70, F.Cu at (149.3, 86.6)
- added DD1: STM32F072RxTx, LQFP_TQFP:LQFP64, F.Cu at (153.1, 126.8)
- added DD2: SX1276, QFN_DFN:QFN-28_EP_6x6_Pitch0.65mm, F.Cu at (150.4, 101.2)
- added L1: 33nH, Inductors:IND_0402, F.Cu at (150.4, 94.3)
- added L2: 2.2nH, Inductors:IND_0402, F.Cu at (148.6, 96.0)
- added L3: 5.6nH, Inductors:IND_0402, F.Cu at (148.6, 91.6)
- added L4: 4.7nH, Inductors:IND_0402, F.Cu at (148.6, 89.4)
- added L5: L, Inductors:IND_0402, F.Cu at (149.3, 81.8)
- added L6: 10nH, Inductors:IND_0402, F.Cu at (155.0, 98.0)
- added L7: Choke, Inductors:IND_0402, F.Cu at (153.2, 106.9)
- added Q1: LED_RGB 5050, LEDs:LED_5050, F.Cu at (163.9, 93.1)
- added R1: 150R, Resistors:RES_0603, F.Cu at (161.2, 116.2)
- added R2: 10k, Resistors:RES_0603, F.Cu at (165.0, 116.2)
- added R3: 10k, Resistors:RES_0603, F.Cu at (163.1, 116.2)
- added R4: 2R0, Resistors:RES_0603, F.Cu at (149.3, 138.4)
- added R5: 1k, Resistors:RES_0603, F.Cu at (153.6, 118.6)
- added R6: 1k, Resistors:RES_0603, F.Cu at (162.3, 98.9)
- added R7: 1k, Resistors:RES_0603, F.Cu at (163.9, 98.9)
- added R8: 1k, Resistors:RES_0603, F.Cu at (165.5, 98.9)
- added R9: 1k, Resistors:RES_0603, F.Cu at (153.5, 85.4)
- added RP1: REFPOINT, PCB:REF_POINT_1MM, F.Cu at (167.4, 139.4)
- added RP2: REFPOINT, PCB:REF_POINT_1MM, F.Cu at (144.0, 83.4)
- added TP1: TESTPOINT, PCB:TESTPOINT_1MM, F.Cu at (146.8, 108.8)
- added TP10: TESTPOINT, PCB:TESTPOINT_1MM, F.Cu at (156.6, 101.2)
- added TP11: TESTPOINT, PCB:TESTPOINT_1MM, F.Cu at (156.6, 99.5)
- added TP2: TESTPOINT, PCB:TESTPOINT_1MM, F.Cu at (148.0, 107.0)
- added TP3: TESTPOINT, PCB:TESTPOINT_1MM, F.Cu at (148.1, 110.9)
- added TP4: TESTPOINT, PCB:TESTPOINT_1MM, F.Cu at (149.3, 108.8)
- added TP5: TESTPOINT, PCB:TESTPOINT_1MM, F.Cu at (150.3, 107.0)
- added TP6: TESTPOINT, PCB:TESTPOINT_1MM, F.Cu at (150.3, 110.9)
- added TP7: TESTPOINT, PCB:TESTPOINT_1MM, F.Cu at (151.9, 108.8)
- added TP8: TESTPOINT, PCB:TESTPOINT_1MM, F.Cu at (156.6, 105.2)
- added TP9: TESTPOINT, PCB:TESTPOINT_1MM, F.Cu at (156.6, 103.1)
- added XL1: CONN_6, Connectors:PLS-6_LOCK, F.Cu at (167.6, 135.0)
- added XL2: CONN_1, Connectors:PLS-1Rnd, F.Cu at (167.6, 116.4)
- added XL3: CONN_5, Connectors:PLS-5, F.Cu at (143.4, 133.6)
- added XL4: CONN_4, Connectors:PBS-4R, F.Cu at (159.3, 108.8)
- added XL5: USB_MICRO_2H, Connectors:USBmicro_MOLEX_1050170001, F.Cu at (155.4, 141.2)
- added XL6: CONN_1, Connectors:PLS-1Rnd, F.Cu at (163.1, 140.1)
- added XTAL1: 12MHz, Quartz:03225C4, F.Cu at (153.8, 116.2)
- added XTAL2: 32MHz, Quartz:03225C4, F.Cu at (144.2, 105.4)
Routing:
- net GND: track 0.00 -> 246.7 mm, vias 0 -> 139
- net +3v3: track 0.00 -> 81.1 mm, vias 0 -> 5
- net VCC: track 0.00 -> 52.1 mm, vias 0 -> 4
- net /RED_LED: track 0.00 -> 35.7 mm, vias 0 -> 2
- net /BLUE_LED: track 0.00 -> 35.7 mm, vias 0 -> 2
- net /GREEN_LED: track 0.00 -> 35.1 mm, vias 0 -> 2
- net /SX_MOSI: track 0.00 -> 31.4 mm, vias 0 -> 2
- net /SX_NSS: track 0.00 -> 31.0 mm, vias 0 -> 2
- net /SX_MISO: track 0.00 -> 28.5 mm, vias 0 -> 2
- net /SX_SCK: track 0.00 -> 26.8 mm, vias 0 -> 2
- net /SDA_PILL: track 0.00 -> 25.3 mm, vias 0 -> 2
- net /SX_DIO5: track 0.00 -> 24.9 mm, vias 0 -> 2
- net /SX_DIO4: track 0.00 -> 23.7 mm, vias 0 -> 2
- net /SX_RST: track 0.00 -> 23.7 mm
- net Net-(DD1-Pad41): track 0.00 -> 21.7 mm, vias 0 -> 1
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- added copper zone on B.Cu, net GND
- added copper zone on F.Cu, net GND
Other:
- board outline added: 27.2 x 86 mm
- copper layers 0 -> 2
