File: UsbHost_hw/UsbHostLora.kicad_pcb (KiCad board)
At the start: 2 copper layers, 27.2 x 86 mm, 78 parts, among them Q1 LED_RGB 5050

Commit message: + GERBERs
Parts:
- added Logo1: Logo, Pictures:Ostranna_16d9_13d5, F.Cu at (154.9, 68.8)
Routing:
- net +3v3: track 81.1 -> 95.2 mm, vias 5 -> 6
- net GND: track 246.7 -> 247.2 mm, vias 139 -> 151
Other:
- board text added: "0"
- board text added: "1"
- board text added: "2"
- board text added: "3"
- board text added: "4"
- board text added: "5"
- board text added: "DBG"
- board text added: "GND"
- board text added: "MISO"
- board text added: "MOSI"
- board text added: "NSS"
- board text added: "Ostranna LoRa UsbHost v1.0"
- board text added: "Rst"
- board text added: "SCK"
