File: UsbHost_hw/UsbHostLora.kicad_sch (KiCad schematic)
At the start: 78 parts

Commit message: sch done
Parts:
- C1, C2, C3, C34, C35: renamed from C?; footprint Capacitors:CAP_0603_Silks -> Capacitors:CAP_0603; Dielectric (none) -> X5R or X7R; Manufacturer (none) -> -; PN (none) -> -; Tolerance (none) -> 20%; Type (none) -> Capacitor SMD; Voltage (none) -> 10V
- C12, C13: renamed from C?; Dielectric (none) -> X5R or X7R; Manufacturer (none) -> -; PN (none) -> -; Tolerance (none) -> 20%; Type (none) -> Capacitor SMD; Voltage (none) -> 10V
- C14, C15, C16, C17, C18, C19, C20, C21, C22, C23, C24, C25, C26, C27, C28, C29, C30, C31, C32, C33: renamed from C?; footprint Capacitors:CAP_0402 -> Capacitors:CAP_0603; Dielectric (none) -> X5R or X7R; Manufacturer (none) -> -; PN (none) -> -; Price (none) -> 0.5; SolderPoints (none) -> 2; Tolerance (none) -> 20%; Type (none) -> Capacitor SMD; Voltage (none) -> 10V
- gave numbers to parts that had none: 51
Connections:
- net +3.3V is gone; now on net +3v3: C13.1, DA1.2 (OUT)
- no-connect marks 7 -> 27
Other:
- moved on the sheet: R1, R2, R3, XL4

Commit message: Routing done
Parts:
- C10, C12, C13, C14, C15, C16, C17, C18, C19, C20, C22, C23, C24, C25, C26, C27, C28, C29, C30, C31, C32, C33, C5, C6, C7, C8, C9: footprint Capacitors:CAP_0603 -> Capacitors:CAP_0402
- C21: value 47pFpF -> 47pF; footprint Capacitors:CAP_0603 -> Capacitors:CAP_0402
- XL3: footprint (none) -> Connectors:PLS-5

Commit message: + GERBERs
Parts:
- added Logo1: Logo, Pictures:Ostranna_16d9_13d5, symbol pcb_details:Logo
Changed lines of the file:
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@@
     (pin "6")
+  )
+  (symbol (lib_id "pcb_details:Logo") (at 317.5 215.9 0) (unit 1)
+    (in_bom yes) (on_board yes) (fields_autoplaced)
+    (property "Reference" "Logo1" (id 0) (at 325.12 214.63 0)
+      (effects (font (size 1.524 1.524)) (justify left))
+    )
+    (property "Value" "Logo" (id 1) (at 325.12 217.17 0)
+      (effects (font (size 1.524 1.524)) (justify left) hide)
+    )
+    (property "Footprint" "Pictures:Ostranna_16d9_13d5" (id 2) (at 317.5 215.9 0)
+      (effects (font (size 1.524 1.524)) hide)
+    )
+    (property "Datasheet" "" (id 3) (at 317.5 215.9 0)
+      (effects (font (size 1.524 1.524)))
+    )
   )
   (symbol (lib_id "Tittar_kl:LED_5050_new") (at 339.09 113.03 0) (unit 1)
@@
       (reference "L7") (unit 1) (value "Choke") (footprint "Inductors:IND_0402")
     )
+    (path "/9be88ee8-c0e9-4c8a-b628-8e5bb8fea86d"
+      (reference "Logo1") (unit 1) (value "Logo") (footprint "Pictures:Ostranna_16d9_13d5")
+    )
     (path "/272bf63d-2c61-4ed5-8c83-046ed99a6be1"

Commit message: + Antenna tuned
Parts:
- C23: value C -> 4.3pF
- C24: value C -> DoNotMount
- L5: value L -> 2.2nH
Changed lines of the file:
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@@
-(kicad_sch (version 20210406) (generator eeschema)
+(kicad_sch (version 20210621) (generator eeschema)
   (paper "A3")
   (junction (at 33.02 85.09) (diameter 1.016) (color 0 0 0 0))
@@
     (in_bom yes) (on_board yes)
     (property "Reference" "L5" (id 0) (at 240.03 226.9236 90))
-    (property "Value" "L" (id 1) (at 240.03 229.235 90))
+    (property "Value" "2.2nH" (id 1) (at 240.03 229.235 90))
     (property "Footprint" "Inductors:IND_0402" (id 2) (at 239.776 230.886 90)
       (effects (font (size 1.016 1.016)) hide)
@@
       (effects (font (size 1.27 1.27)) (justify left))
     )
-    (property "Value" "C" (id 1) (at 229.87 236.22 0)
+    (property "Value" "4.3pF" (id 1) (at 229.87 236.22 0)
       (effects (font (size 1.27 1.27)) (justify left))
     )
@@
       (effects (font (size 1.27 1.27)) (justify left))
     )
-    (property "Value" "C" (id 1) (at 245.11 236.22 0)
+    (property "Value" "DoNotMount" (id 1) (at 241.3 236.22 0)
       (effects (font (size 1.27 1.27)) (justify left))
     )
@@
     )
     (path "/dc69873b-38e2-47b6-baef-31c68bc4c2cd"
-      (reference "C23") (unit 1) (value "C") (footprint "Capacitors:CAP_0402")
+      (reference "C23") (unit 1) (value "4.3pF") (footprint "Capacitors:CAP_0402")
     )
     (path "/7ff32c8e-447d-4509-9d42-6d840dfd1e25"
-      (reference "C24") (unit 1) (value "C") (footprint "Capacitors:CAP_0402")
+      (reference "C24") (unit 1) (value "DoNotMount") (footprint "Capacitors:CAP_0402")
     )
     (path "/252132bb-e3df-450e-9d85-b98b5fa4beb8"
@@
     )
     (path "/d663e092-b7e2-4a8e-a057-8a63ed211d7e"
-      (reference "L5") (unit 1) (value "L") (footprint "Inductors:IND_0402")
+      (reference "L5") (unit 1) (value "2.2nH") (footprint "Inductors:IND_0402")
     )
     (path "/c9d3d319-421a-4e5b-bf6c-da7f6ea3ca68"

Commit message: Release
Parts:
- C34, C35: value 18pF -> 10pF
Changed lines of the file:
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@@
       (effects (font (size 1.27 1.27)) (justify left))
     )
-    (property "Value" "18pF" (id 1) (at 111.76 278.13 0)
+    (property "Value" "10pF" (id 1) (at 111.76 278.13 0)
       (effects (font (size 1.27 1.27)) (justify left))
     )
@@
       (effects (font (size 1.27 1.27)) (justify left))
     )
-    (property "Value" "18pF" (id 1) (at 127 278.13 0)
+    (property "Value" "10pF" (id 1) (at 127 278.13 0)
       (effects (font (size 1.27 1.27)) (justify left))
     )
@@
     )
     (path "/ba3cbddd-b2b3-4fb3-a4c0-21fdcc08cb98"
-      (reference "C34") (unit 1) (value "18pF") (footprint "Capacitors:CAP_0603")
+      (reference "C34") (unit 1) (value "10pF") (footprint "Capacitors:CAP_0603")
     )
     (path "/4285ac09-5692-4e40-bbb4-97d0b6ed77ba"
-      (reference "C35") (unit 1) (value "18pF") (footprint "Capacitors:CAP_0603")
+      (reference "C35") (unit 1) (value "10pF") (footprint "Capacitors:CAP_0603")
     )
     (path "/07ee0de6-6063-409b-83b9-51169694bd72"
