File: UsbHost_hw/UsbHostLora.kicad_sch (KiCad schematic)
At the start: 79 parts, among them Q1 LED_RGB 5050

Commit message: Sent to factory
Parts:
- removed ANT1: ANT_PCB_MONO_2PIN, Antennas:Firefly_868, symbol Antennas_kl:ANT_PCB_MONO
- removed C10, C28, C29, C30, C32, C33: 0.1u, Capacitors:CAP_0402, symbol Tittar_kl:C
- removed C11: 1u, Capacitors:CAP_0603, symbol Tittar_kl:C
- removed C16: 1.5pF, Capacitors:CAP_0402, symbol Tittar_kl:C
- removed C17: 22pF, Capacitors:CAP_0402, symbol Tittar_kl:C
- removed C18, C19: 8.2pF, Capacitors:CAP_0402, symbol Tittar_kl:C
- removed C20, C25: 3.3pF, Capacitors:CAP_0402, symbol Tittar_kl:C
- removed C21, C22, C31: 47pF, Capacitors:CAP_0402, symbol Tittar_kl:C
- removed C23: 4.3pF, Capacitors:CAP_0402, symbol Tittar_kl:C
- removed C24: DoNotMount, Capacitors:CAP_0402, symbol Tittar_kl:C
- removed C26, C27: 1000pF, Capacitors:CAP_0402, symbol Tittar_kl:C
- removed C34, C35: 10pF, Capacitors:CAP_0603, symbol Tittar_kl:C
- removed DA1: MCP1700, SOT:SOT23-3A, symbol Power_kl:MCP1700
- removed DA2: PE4259, SOT:SC70, symbol RF_ICs:PE4259
- removed DD1: STM32F072RxTx, LQFP_TQFP:LQFP64, symbol st_kl:STM32F072RxTx
- removed DD2: SX1276, QFN_DFN:QFN-28_EP_6x6_Pitch0.65mm, symbol RF_ICs:SX1276
- removed L4: 4.7nH, Inductors:IND_0402, symbol Tittar_kl:L
- removed L5: 2.2nH, Inductors:IND_0402, symbol Tittar_kl:L
- removed L6: 10nH, Inductors:IND_0402, symbol Tittar_kl:L
- removed L7: Choke, Inductors:IND_0402, symbol Tittar_kl:L
- removed Q1: LED_RGB 5050, LEDs:LED_5050, symbol Tittar_kl:LED_5050_new
- removed TP10, TP11: TESTPOINT, PCB:TESTPOINT_1MM, symbol pcb_details:TESTPOINT
- removed XL1: CONN_6, Connectors:PLS-6_LOCK, symbol Connectors_kl:CONN_6
- removed XL2, XL6: CONN_1, Connectors:PLS-1Rnd, symbol Connectors_kl:CONN_1
- removed XL3: CONN_5, Connectors:PLS-5, symbol Connectors_kl:CONN_5
- removed XL4: CONN_4, Connectors:PBS-4R, symbol Connectors_kl:CONN_4
- removed XL5: USB_MICRO_2H, Connectors:USBmicro_MOLEX_1050170001, symbol Connectors_kl:USB_MICRO_2H
- removed XTAL1: 12MHz, Quartz:03225C4, symbol Tittar_kl:CRYSTAL_H
- removed XTAL2: 32MHz, Quartz:03225C4, symbol Tittar_kl:CRYSTAL_H
- added DA1: CJ6101B33M, SOT:SOT23-5, symbol Power_kl:LDO_5pin_4NC
- added DD1: GD32E103CB, LQFP_TQFP:LQFP48, symbol GD:GD32E103CB
- added MDL1: E220-900MM22S, Modules:E220-900MM22S, symbol RF_ICs:E220-900MM22S
- added Q1, Q2: LED_5050, LEDs:LED_5050, symbol LEDs:LED_5050
- added XL1: SOCKET_6, Connectors:PLS-6_LOCK, symbol Connectors_kl:SOCKET_6
- added XL2: DS1144-18-16FS8BNR0, Connectors:USBC_10PF-074_1, symbol Connectors_kl:USBC-16P
- added XL3: SOCKET_5, Connectors:PLS-5, symbol Connectors_kl:SOCKET_5
- added XL4: CONN_1, PCB:OSCIL_GND, symbol Connectors_kl:CONN_1
- added XL5: SMA_L, Connectors:SMA_R, symbol Connectors_kl:SMA_L
- C1: value 2u2 -> 1u; footprint Capacitors:CAP_0603 -> Capacitors:CAP_0603_Silks; Dielectric X5R or X7R -> (none); Manufacturer - -> (none); Price 0.5 -> (none); SolderPoints 2 -> (none); Type Capacitor SMD -> (none); URL (none) -> -
- C12: value 0.1u -> 10nF; footprint Capacitors:CAP_0402 -> Capacitors:CAP_0603_Silks; Dielectric X5R or X7R -> (none); Manufacturer - -> (none); Price 0.5 -> (none); SolderPoints 2 -> (none); Type Capacitor SMD -> (none); URL (none) -> -
- C13, C6: value 0.1u -> 10u; footprint Capacitors:CAP_0402 -> Capacitors:CAP_0603_Silks; Dielectric X5R or X7R -> (none); Manufacturer - -> (none); Price 0.5 -> (none); SolderPoints 2 -> (none); Type Capacitor SMD -> (none); URL (none) -> -
- C14: value 10n -> DNM; footprint Capacitors:CAP_0402 -> Capacitors:CAP_0402_Silks; Dielectric X5R or X7R -> (none); Manufacturer - -> (none); Price 0.5 -> (none); SolderPoints 2 -> (none); Type Capacitor SMD -> (none); URL (none) -> -
- C15: value 47pF -> DNM; footprint Capacitors:CAP_0402 -> Capacitors:CAP_0402_Silks; Dielectric X5R or X7R -> (none); Manufacturer - -> (none); Price 0.5 -> (none); SolderPoints 2 -> (none); Type Capacitor SMD -> (none); URL (none) -> -
- C2: value 18pF -> 2u2; footprint Capacitors:CAP_0603 -> Capacitors:CAP_0603_Silks; Dielectric X5R or X7R -> (none); Manufacturer - -> (none); Price 0.5 -> (none); SolderPoints 2 -> (none); Type Capacitor SMD -> (none); URL (none) -> -
- C3: value 18pF -> 1u; footprint Capacitors:CAP_0603 -> Capacitors:CAP_0603_Silks; Dielectric X5R or X7R -> (none); Manufacturer - -> (none); Price 0.5 -> (none); SolderPoints 2 -> (none); Type Capacitor SMD -> (none); URL (none) -> -
- C4: value 10u -> 1u; footprint Capacitors:CAP_0603 -> Capacitors:CAP_0603_Silks; Dielectric X5R or X7R -> (none); Manufacturer - -> (none); Price 0.5 -> (none); SolderPoints 2 -> (none); Type Capacitor SMD -> (none); URL (none) -> -
- C5: value 0.1u -> 10n; footprint Capacitors:CAP_0402 -> Capacitors:CAP_0603_Silks; Dielectric X5R or X7R -> (none); Manufacturer - -> (none); Price 0.5 -> (none); SolderPoints 2 -> (none); Type Capacitor SMD -> (none); URL (none) -> -
- C7, C8, C9: footprint Capacitors:CAP_0402 -> Capacitors:CAP_0603_Silks; Dielectric X5R or X7R -> (none); Manufacturer - -> (none); Price 0.5 -> (none); SolderPoints 2 -> (none); Type Capacitor SMD -> (none); URL (none) -> -
- L1: value 33nH -> 330nH; PN (none) -> -; Tolerance (none) -> 20%; Type (none) -> Inductor SMD
- L2: value 2.2nH -> BLM15AG102SN1; PN (none) -> -; Tolerance (none) -> 20%; Type (none) -> Inductor SMD
- L3: value 5.6nH -> 0R; PN (none) -> -; Tolerance (none) -> 20%; Type (none) -> Inductor SMD
- Logo1: footprint Pictures:Ostranna_16d9_13d5 -> Pictures:Ostranna_12d7_10d1
- R1: value 150R -> 2R0; footprint Resistors:RES_0603 -> Resistors:RES_0603_RefFab; PN (none) -> -; Price 0.5 -> (none); SolderPoints 2 -> (none); Tolerance (none) -> 1%
- R2, R3: value 10k -> 5k1; footprint Resistors:RES_0603 -> Resistors:RES_0603_RefFab; PN (none) -> -; Price 0.5 -> (none); SolderPoints 2 -> (none); Tolerance (none) -> 1%
- R4: value 2R0 -> 1k; footprint Resistors:RES_0603 -> Resistors:RES_0603_RefFab; PN (none) -> -; Price 0.5 -> (none); SolderPoints 2 -> (none); Tolerance (none) -> 1%
- R5, R6, R7, R8, R9: footprint Resistors:RES_0603 -> Resistors:RES_0603_RefFab; PN (none) -> -; Price 0.5 -> (none); SolderPoints 2 -> (none); Tolerance (none) -> 1%
- RP1, RP2: Price 0 -> (none); SolderPoints 0 -> (none)
Connections:
- net PWR_PILL_PROT is gone; now on an unnamed net: R1.2
- net SCL_PILL is gone; now on net GND: R3.2
- net +3v3: now also C3.1, L2.1, DA1.5 (OUT), DD1.1 (VBAT), DD1.24 (VDD1), DD1.36 (VDD2), DD1.48 (VDD3), DD1.9 (VDDA), XL1.1, XL3.5; no longer C13.1
- net GND: now also L1.1, R2.1, DA1.2 (GND), DA1.4 (NC), DD1.23 (VSS1), DD1.35 (VSS2), DD1.44 (BOOT0), DD1.47 (VSS3), DD1.8 (VSSA), MDL1.16 (GND), MDL1.2 (GND), MDL1.7 (GND), Q1.4 (B), Q1.5 (G), Q1.6, Q2.4 (B), Q2.5 (G), Q2.6, XL1.3, XL2.A1B12 (GND), XL2.B1A12 (GND), XL3.1, XL4.1 (P1), XL5.GND
- net SWCLK: now also DD1.37 (SWCLK), XL1.2
- net SWDIO: now also DD1.34 (SWDIO), XL1.4
- net UART_RX: now also DD1.31 (PA10), XL1.6
- net UART_TX: now also DD1.30 (PA9), XL1.5
- net at R4.2: now also Q1.1; no longer C1.1
- net LED1_R: now reaches R5.1
- net LED1_R: now also DD1.39 (JTDO); no longer C3.1
- net at R5.2: now also Q1.2
- net at R8.2: now also Q2.2
- net at R6.2: now also Q1.3
- net at R7.2: now also Q2.1
- net ANT3: now reaches L3.2
- net ANT3: now also C14.1, L1.2, MDL1.6 (ANT)
- net +R_PWR: now reaches L2.2
- net +R_PWR: now also C12.1, C13.1, MDL1.1 (VCC); no longer L1.2
- net LED2_G: now reaches R9.1
- net LED2_G: now also DD1.27 (PB14)
- net at L3.1: now also C15.1, XL5.RF
- net at R9.2: now also Q2.3
- net 5V_USB renamed LED1_B
- net LED1_B: now also DD1.22 (PB11); no longer C12.1
- net BLUE_LED renamed LED2_R
- net LED2_R: now also DD1.19 (PB1)
- net GREEN_LED renamed LED1_G
- net LED1_G: now also DD1.21 (PB10)
- removed net PWR_PILL: R1.1, R2.1, R3.1
- net RED_LED renamed LED2_B
- net LED2_B: now also DD1.18 (PB0)
- net SDA_PILL: no longer names the net of R2.2
- net SDA_PILL: now also XL2.A5 (CC1)
- net SX_DIO0 renamed R_DIO3
- net R_DIO3: now also DD1.11 (PA1), MDL1.18 (DIO3)
- net SX_DIO1 renamed R_BUSY
- net R_BUSY: now also DD1.12 (PA2), MDL1.11 (BUSY)
- net SX_DIO2 renamed R_RXEN
- net R_RXEN: now also DD1.13 (PA3), MDL1.10 (RXEN)
- net SX_DIO3 renamed R_NSS
- net R_NSS: now also DD1.14 (PA4), MDL1.14 (NSS)
- net SX_DIO4 renamed R_SCK
- net R_SCK: now also DD1.15 (PA5), MDL1.15 (SCK)
- net SX_DIO5 renamed R_MISO
- net R_MISO: now also DD1.16 (PA6), MDL1.12 (MISO)
- net SX_MISO renamed R_RST
- net R_RST: now also DD1.29 (PA8), MDL1.3 (NRST)
- net SX_RST renamed R_DIO1
- net R_DIO1: now also DD1.10 (PA0), MDL1.20 (DIO1)
- net SX_SCK renamed R_MOSI
- net R_MOSI: now also DD1.17 (PA7), MDL1.13 (MOSI)
- new net: R3.1, XL2.B5 (CC2)
- new net: MDL1.19 (DIO2), MDL1.9 (TXEN)
- new net +5vUSB: C1.1, DA1.1 (IN), DA1.3 (EN), R1.1, XL2.A4B9 (VBUS), XL2.B4A9 (VBUS)
- new net PB6: DD1.42 (PB6), XL3.2
- new net PB7: DD1.43 (PB7), XL3.3
- new net PB8: DD1.45 (PB8), XL3.4
- new net USB.DN: DD1.32 (PA11), XL2.A7 (DN1), XL2.B7 (DN2)
- new net USB.DP: DD1.33 (PA12), XL2.A6 (DP1), XL2.B6 (DP2)
- no-connect marks 27 -> 20
Other:
- note added: "Just Pins"
- note added: "NC is connected to GND to improve thermal performance"
- note removed: "DEBUG pin"
- note removed: "LORA"
- note removed: "Peripheral I2C Pull-Ups"
- note removed: "Pill"
- note removed: "Pill Connector"
- note removed: "RGB LED"
